File: controller/Stratosensor.sch (KiCad schematic (older format))
At the start: 34 parts, among them J1 ISP, J10 A45, J11 A67, J2 BME280, J3 BME280, J4 UART, J5 POWER, J6 I2C, J7 I2C, J8 A01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

Commit message: Revision 2 of controller board
Signed-off-by: Alexey Galakhov <agalakhov@gmail.com>
Parts:
- C1, C2: footprint Capacitor_THT:C_Rect_L4.0mm_W2.5mm_P2.50mm -> Capacitor_THT:C_Disc_D4.7mm_W2.5mm_P5.00mm
- U1: symbol MCU_Microchip_ATmega:ATmega1284-PU -> Stratosensor-rescue:ATmega1284-PU-MCU_Microchip_ATmega
Changed lines of the file:
@@
 EESchema Schematic File Version 4
 LIBS:Stratosensor-cache
-EELAYER 29 0
+EELAYER 30 0
 EELAYER END
 $Descr A4 11693 8268
@@
 F 0 "C1" V 1098 2300 50  0000 C CNN
 F 1 "12p" V 1189 2300 50  0000 C CNN
-F 2 "Capacitor_THT:C_Rect_L4.0mm_W2.5mm_P2.50mm" H 1388 2150 50  0001 C CNN
+F 2 "Capacitor_THT:C_Disc_D4.7mm_W2.5mm_P5.00mm" H 1388 2150 50  0001 C CNN
 F 3 "~" H 1350 2300 50  0001 C CNN
 	1    1350 2300
@@
 F 0 "C2" V 1500 2600 50  0000 C CNN
 F 1 "12p" V 1600 2600 50  0000 C CNN
-F 2 "Capacitor_THT:C_Rect_L4.0mm_W2.5mm_P2.50mm" H 1388 2450 50  0001 C CNN
+F 2 "Capacitor_THT:C_Disc_D4.7mm_W2.5mm_P5.00mm" H 1388 2450 50  0001 C CNN
 F 3 "~" H 1350 2600 50  0001 C CNN
 	1    1350 2600
@@
 Connection ~ 6800 4650
 $Comp
-L MCU_Microchip_ATmega:ATmega1284-PU U1
+L Stratosensor-rescue:ATmega1284-PU-MCU_Microchip_ATmega U1
 U 1 1 5D4D949A
 P 2700 3850
@@
 	8350 2050 8350 1650
 Wire Bus Line
-	8350 1650 7350 1650
-Wire Bus Line
 	7350 1650 7350 1350
 Wire Bus Line
 	7350 1350 3700 1350
-Wire Bus Line
-	8450 4150 8450 4650
-Wire Bus Line
-	6800 4650 6800 5150
-Wire Bus Line
-	4450 4050 4450 4600
-Wire Bus Line
-	6650 4150 6650 4600
-Wire Bus Line
-	5150 4150 5150 4600
-Wire Bus Line
-	9400 1300 9400 1950
-Wire Bus Line
-	10100 1300 10100 2050
-Wire Bus Line
-	8650 1300 8650 1950
-Wire Bus Line
-	7900 1300 7900 1550
-Wire Bus Line
-	8350 2050 10100 2050
-Wire Bus Line
-	6150 2400 6150 3000
-Wire Bus Line
-	4100 2150 4100 2700
-Wire Bus Line
-	3750 3000 3750 3650
-Wire Bus Line
-	3700 1350 3700 2750
 Entry Bus Bus
 	7800 1650 7900 1550
+Wire Bus Line
+	7350 1650 8350 1650
+Wire Bus Line
+	8450 4150 8450 4650
+Wire Bus Line
+	6800 4650 6800 5150
+Wire Bus Line
+	4450 4050 4450 4600
+Wire Bus Line
+	6650 4150 6650 4600
+Wire Bus Line
+	5150 4150 5150 4600
+Wire Bus Line
+	9400 1300 9400 1950
+Wire Bus Line
+	10100 1300 10100 2050
+Wire Bus Line
+	8650 1300 8650 1950
+Wire Bus Line
+	7900 1300 7900 1550
+Wire Bus Line
+	8350 2050 10100 2050
+Wire Bus Line
+	6150 2400 6150 3000
+Wire Bus Line
+	4100 2150 4100 2700
+Wire Bus Line
+	3750 3000 3750 3650
+Wire Bus Line
+	3700 1350 3700 2750
 $EndSCHEMATC
