File: stratosensor-power/stratosensor-power.kicad_pcb (KiCad board)
At the start: 2 copper layers, 100 x 100 mm, 59 parts, among them J1 OUT, J2 OUT, J3 OUT, U1 AP65111AWU, U2 AP65111AWU, U3 AP65111AWU

Commit message: Finish power board
Signed-off-by: Alexey Galakhov <agalakhov@gmail.com>
Parts:
- added G***: LOGO, ublox:logo2_front, B.Cu at (129.7, 100.0)
- added G***: LOGO, ublox:logo, B.Cu at (152.5, 100.0)
- added REF**: MountingHole_3.2mm_M3_DIN965, MountingHole:MountingHole_3.2mm_M3_DIN965, F.Cu at (124.6, 143.2)
- added REF**: MountingHole_3.2mm_M3_DIN965, MountingHole:MountingHole_3.2mm_M3_DIN965, F.Cu at (160.2, 143.2)
- added REF**: MountingHole_3.2mm_M3_DIN965, MountingHole:MountingHole_3.2mm_M3_DIN965, F.Cu at (160.2, 56.8)
- added REF**: MountingHole_3.2mm_M3_DIN965, MountingHole:MountingHole_3.2mm_M3_DIN965, F.Cu at (124.6, 56.8)
Routing:
- net GND: vias 18 -> 21
Other:
- board text added: "-"
- board text added: "Gymnasium Brake Project Stratosphere 09-2019"

Commit message: Finish and generate gerbers
Signed-off-by: Alexey Galakhov <agalakhov@snapview.de>
Parts:
- added J4: TP-, Connector_PinHeader_2.54mm:PinHeader_1x01_P2.54mm_Vertical, F.Cu at (114.4, 143.2)
- added J5: TP+, Connector_PinHeader_2.54mm:PinHeader_1x01_P2.54mm_Vertical, F.Cu at (114.4, 56.8)
- BT1, BT2, BT3: footprint Battery:BatteryHolder_MPD_BH-18650-PC2 -> bat:BatteryHolder_COMF_BHC-18650-1
- F1, F3: value 85°C -> 84°C; footprint Resistor_THT:R_Axial_Power_L20.0mm_W6.4mm_P25.40mm -> Resistor_THT:R_Axial_DIN0411_L9.9mm_D3.6mm_P25.40mm_Horizontal
- F2, F4: value 3.15A -> 3.5A; footprint Resistor_THT:R_Axial_Power_L20.0mm_W6.4mm_P25.40mm -> Resistor_THT:R_Axial_DIN0309_L9.0mm_D3.2mm_P15.24mm_Horizontal
- moved BT1 90.4 mm to (176.7, 127.9), turned to 180 degrees
- moved BT3 90.4 mm to (176.7, 72.1), turned to 180 degrees
- moved BT2 71.1 mm to (176.7, 100.0), turned to 180 degrees
- moved F1 58.0 mm to (119.5, 114.0), turned to 0 degrees
- moved F3 58.0 mm to (119.5, 86.0), turned to 0 degrees
- moved F2 29.7 mm to (150.0, 114.0), turned to 0 degrees
- moved F4 29.7 mm to (150.0, 86.0), turned to 0 degrees
- moved G*** 29.7 mm to (139.8, 127.9), turned to 180 degrees
- moved G*** 25.6 mm to (141.1, 77.1), turned to 180 degrees
Routing:
- net Net-(BT2-Pad2): track 17.0 -> 20.0 mm
- net Net-(BT1-Pad2): track 17.0 -> 20.0 mm
- net Net-(BT3-Pad1): track 17.7 -> 20.2 mm
- net Net-(BT2-Pad1): track 17.7 -> 20.2 mm
- net VDC: vias 27 -> 40
- net GND: vias 21 -> 27
Other:
- rule pad_to_mask_clearance: 0.051 -> 0.02
- rule solder_mask_min_width: 0.25 -> 0.2
- board text added: "3x 3.7V 18650 Li-Ion Unprotected Output 3x 3.3/5V 1A"
- board text added: "V"
