File: stratosensor-power/stratosensor-power.sch (KiCad schematic (older format))
At the start: 55 parts, among them J1 OUT, J2 OUT, J3 OUT, U1 AP65111AWU, U2 AP65111AWU, U3 AP65111AWU

Commit message: Finish and generate gerbers
Signed-off-by: Alexey Galakhov <agalakhov@snapview.de>
Parts:
- added J4: TP-, Connector_PinHeader_2.54mm:PinHeader_1x01_P2.54mm_Vertical, symbol Connector:Conn_01x01_Male
- added J5: TP+, Connector_PinHeader_2.54mm:PinHeader_1x01_P2.54mm_Vertical, symbol Connector:Conn_01x01_Male
- BT1, BT2, BT3: footprint Battery:BatteryHolder_MPD_BH-18650-PC2 -> bat:BatteryHolder_COMF_BHC-18650-1
- F1, F3: value 85°C -> 84°C; footprint Resistor_THT:R_Axial_Power_L20.0mm_W6.4mm_P25.40mm -> Resistor_THT:R_Axial_DIN0411_L9.9mm_D3.6mm_P25.40mm_Horizontal
- F2, F4: value 3.15A -> 3.5A; footprint Resistor_THT:R_Axial_Power_L20.0mm_W6.4mm_P25.40mm -> Resistor_THT:R_Axial_DIN0309_L9.0mm_D3.2mm_P15.24mm_Horizontal
Connections:
- net GND: now also J4.1 (Pin_1)
- net VDC: now also J5.1 (Pin_1)
Changed lines of the file:
@@
 F 0 "BT3" H 1418 5146 50  0000 L CNN
 F 1 "18650" H 1418 5055 50  0000 L CNN
-F 2 "Battery:BatteryHolder_MPD_BH-18650-PC2" V 1300 5110 50  0001 C CNN
+F 2 "bat:BatteryHolder_COMF_BHC-18650-1" V 1300 5110 50  0001 C CNN
 F 3 "~" V 1300 5110 50  0001 C CNN
 	1    1300 5050
@@
 F 0 "BT2" H 1418 4246 50  0000 L CNN
 F 1 "18650" H 1418 4155 50  0000 L CNN
-F 2 "Battery:BatteryHolder_MPD_BH-18650-PC2" V 1300 4210 50  0001 C CNN
+F 2 "bat:BatteryHolder_COMF_BHC-18650-1" V 1300 4210 50  0001 C CNN
 F 3 "~" V 1300 4210 50  0001 C CNN
 	1    1300 4150
@@
 F 0 "BT1" H 1418 3346 50  0000 L CNN
 F 1 "18650" H 1418 3255 50  0000 L CNN
-F 2 "Battery:BatteryHolder_MPD_BH-18650-PC2" V 1300 3310 50  0001 C CNN
+F 2 "bat:BatteryHolder_COMF_BHC-18650-1" V 1300 3310 50  0001 C CNN
 F 3 "~" V 1300 3310 50  0001 C CNN
 	1    1300 3250
@@
 P 1300 3800
 F 0 "F2" H 1360 3846 50  0000 L CNN
-F 1 "3.15A" H 1360 3755 50  0000 L CNN
-F 2 "Resistor_THT:R_Axial_Power_L20.0mm_W6.4mm_P25.40mm" V 1230 3800 50  0001 C CNN
+F 1 "3.5A" H 1360 3755 50  0000 L CNN
+F 2 "Resistor_THT:R_Axial_DIN0309_L9.0mm_D3.2mm_P15.24mm_Horizontal" V 1230 3800 50  0001 C CNN
 F 3 "~" H 1300 3800 50  0001 C CNN
 	1    1300 3800
@@
 P 1300 4400
 F 0 "F3" H 1388 4446 50  0000 L CNN
-F 1 "85°C" H 1388 4355 50  0000 L CNN
-F 2 "Resistor_THT:R_Axial_Power_L20.0mm_W6.4mm_P25.40mm" H 1350 4200 50  0001 L CNN
+F 1 "84°C" H 1388 4355 50  0000 L CNN
+F 2 "Resistor_THT:R_Axial_DIN0411_L9.9mm_D3.6mm_P25.40mm_Horizontal" H 1350 4200 50  0001 L CNN
 F 3 "~" H 1300 4400 50  0001 C CNN
 	1    1300 4400
@@
 P 1300 4700
 F 0 "F4" H 1360 4746 50  0000 L CNN
-F 1 "3.15A" H 1360 4655 50  0000 L CNN
-F 2 "Resistor_THT:R_Axial_Power_L20.0mm_W6.4mm_P25.40mm" V 1230 4700 50  0001 C CNN
+F 1 "3.5A" H 1360 4655 50  0000 L CNN
+F 2 "Resistor_THT:R_Axial_DIN0309_L9.0mm_D3.2mm_P15.24mm_Horizontal" V 1230 4700 50  0001 C CNN
 F 3 "~" H 1300 4700 50  0001 C CNN
 	1    1300 4700
@@
 P 1300 3500
 F 0 "F1" H 1388 3546 50  0000 L CNN
-F 1 "85°C" H 1388 3455 50  0000 L CNN
-F 2 "Resistor_THT:R_Axial_Power_L20.0mm_W6.4mm_P25.40mm" H 1350 3300 50  0001 L CNN
+F 1 "84°C" H 1388 3455 50  0000 L CNN
+F 2 "Resistor_THT:R_Axial_DIN0411_L9.9mm_D3.6mm_P25.40mm_Horizontal" H 1350 3300 50  0001 L CNN
 F 3 "~" H 1300 3500 50  0001 C CNN
 	1    1300 3500
 	1    0    0    -1
 $EndComp
+$Comp
+L Connector:Conn_01x01_Male J5
+U 1 1 5D944DE5
+P 1900 3050
+F 0 "J5" H 1872 2982 50  0000 R CNN
+F 1 "TP+" H 1872 3073 50  0000 R CNN
+F 2 "Connector_PinHeader_2.54mm:PinHeader_1x01_P2.54mm_Vertical" H 1900 3050 50  0001 C CNN
+F 3 "~" H 1900 3050 50  0001 C CNN
+	1    1900 3050
+	-1   0    0    1
+$EndComp
+$Comp
+L Connector:Conn_01x01_Male J4
+U 1 1 5D9468D8
+P 1900 5150
+F 0 "J4" H 1872 5082 50  0000 R CNN
+F 1 "TP-" H 1872 5173 50  0000 R CNN
+F 2 "Connector_PinHeader_2.54mm:PinHeader_1x01_P2.54mm_Vertical" H 1900 5150 50  0001 C CNN
+F 3 "~" H 1900 5150 50  0001 C CNN
+	1    1900 5150
+	-1   0    0    1
+$EndComp
+Wire Wire Line
+	1300 3050 1700 3050
+Wire Wire Line
+	1300 5150 1700 5150
 $EndSCHEMATC
